File: anode-driver.sch (KiCad schematic (older format))
At the start: 48 parts

Commit message: I think the layout is finished now. I'll check again after I sleep.
Parts:
- Q1, Q10, Q11, Q12, Q13, Q14, Q15, Q16, Q2, Q3, Q4, Q5, Q6, Q7, Q8, Q9: renamed from Q?; footprint SOT-23 -> Housings_SOT-23_SOT-143_TSOT-6:SOT-23
- R24, R25, R26, R27, R28, R29, R30, R31, R32, R33, R34, R35, R36, R37, R38, R39, R40, R41, R42, R43, R44, R45, R46, R47, R48, R49, R50, R51, R52, R53, R54, R55: renamed from R?; footprint (none) -> Resistors_SMD:R_0603; symbol R -> R-RESCUE-score-module-pcb-v1
Connections:
- net ANODE0_DRV: now also Q3.3 (C); no longer Q3.2 (E)
- net ANODE1_DRV: now also Q7.3 (C); no longer Q7.2 (E)
- net ANODE2: now also R40.2
- net ANODE2_DRV: now also Q11.3 (C); no longer Q11.2 (E)
- net ANODE3_DRV: now also Q15.3 (C); no longer Q15.2 (E)
- net ANODE4_DRV: now also Q4.3 (C); no longer Q4.2 (E)
- net ANODE5_DRV: now also Q8.3 (C); no longer Q8.2 (E)
- net ANODE6_DRV: now also Q12.3 (C); no longer Q12.2 (E)
- net ANODE7_DRV: now also Q16.3 (C); no longer Q16.2 (E)
- net DISPLAY_5V: now also Q11.2 (E), Q12.2 (E), Q15.2 (E), Q16.2 (E), Q3.2 (E), Q4.2 (E), Q7.2 (E), Q8.2 (E); no longer Q11.3 (C), Q12.3 (C), Q15.3 (C), Q16.3 (C), Q3.3 (C), Q4.3 (C), Q7.3 (C), Q8.3 (C)
