File: cathode-driver.sch (KiCad schematic (older format))
At the start: 40 parts

Commit message: I think the layout is finished now. I'll check again after I sleep.
Parts:
- removed Q? (x4): BC846, SOT-23, symbol BC846
- removed R? (x4): 120, symbol R
- added Q33: BC846, Housings_SOT-23_SOT-143_TSOT-6:SOT-23, symbol BC846
- added R72: 120, Resistors_SMD:R_0603, symbol R-RESCUE-score-module-pcb-v1
- Q17, Q18, Q19, Q20, Q21, Q22, Q23, Q24, Q25, Q26, Q27, Q28, Q29, Q30, Q31, Q32: renamed from Q?; footprint SOT-23 -> Housings_SOT-23_SOT-143_TSOT-6:SOT-23
- R56, R57, R58, R59, R60, R61, R62, R63, R64, R65, R66, R67, R68, R69, R70, R71: renamed from R?; footprint (none) -> Resistors_SMD:R_0603; symbol R -> R-RESCUE-score-module-pcb-v1
Connections:
- net CATHODE16: now also Q33.1 (B)
- net CATHODE16_DRV: now also Q33.3 (C)
- net GND: now also R72.2
- new net: Q33.2 (E), R72.1
