File: power-supply.sch (KiCad schematic (older format))
At the start: 27 parts, among them U5 AP3513E, U7 AP1117IE33G

Commit message: I think the layout is finished now. I'll check again after I sleep.
Parts:
- C10: renamed from C16; symbol CP -> CP-RESCUE-score-module-pcb-v1
- C11: renamed from C17; symbol CP -> CP-RESCUE-score-module-pcb-v1
- C12: renamed from C20; symbol CP -> CP-RESCUE-score-module-pcb-v1
- C13: renamed from C12; symbol C -> C-RESCUE-score-module-pcb-v1
- C14: renamed from C18; symbol C -> C-RESCUE-score-module-pcb-v1
- C15: renamed from C19; symbol C -> C-RESCUE-score-module-pcb-v1
- C16: renamed from C13; symbol C -> C-RESCUE-score-module-pcb-v1
- C17: renamed from C14; symbol CP -> CP-RESCUE-score-module-pcb-v1
- C18: renamed from C15; symbol CP -> CP-RESCUE-score-module-pcb-v1
- C19: renamed from C21; symbol CP -> CP-RESCUE-score-module-pcb-v1
- C20: renamed from C22; symbol C -> C-RESCUE-score-module-pcb-v1
- L1: footprint Inductors:SELF-WE-PD-XXL -> Inductors:SELF-WE-PD3S
- R15: renamed from R37; symbol R -> R-RESCUE-score-module-pcb-v1
- R16: renamed from R38; symbol R -> R-RESCUE-score-module-pcb-v1
- R17: renamed from R33; symbol R -> R-RESCUE-score-module-pcb-v1
- R18: renamed from R34; symbol R -> R-RESCUE-score-module-pcb-v1
- R19: renamed from R35; symbol R -> R-RESCUE-score-module-pcb-v1
- R20: renamed from R31; symbol R -> R-RESCUE-score-module-pcb-v1
- R21: renamed from R39; symbol R -> R-RESCUE-score-module-pcb-v1
- R22: renamed from R40; symbol R -> R-RESCUE-score-module-pcb-v1
- R23: renamed from R41; symbol R -> R-RESCUE-score-module-pcb-v1
- renumbered U5 to U3, U7 to U4
Connections:
- net GND: now also D1.1 (K), D2.1 (K), D3.1 (K); no longer D1.2 (A), D2.2 (A), D3.2 (A)
- net at R21.2: now also D1.2 (A); no longer D1.1 (K)
- net at R22.2: now also D2.2 (A); no longer D2.1 (K)
- net at R23.2: now also D3.2 (A); no longer D3.1 (K)
