File: score-module-pcb-v1.kicad_pcb (KiCad board)
At the start: 4 copper layers, 199.7 x 64.8 mm, 159 parts, among them P1 PINBALL-CONNECTOR, P2 PINBALL-CONNECTOR, Q1 BC846, Q10 BC846, Q11 BC856, Q12 BC856, Q13 BC846, Q14 BC846, Q15 BC856, Q16 BC856, Q17 BC846, Q18 BC846, Q19 BC846, Q2 BC846, Q20 BC846, Q21 BC846, Q22 BC846, Q23 BC846, Q24 BC846, Q25 BC846, Q26 BC846, Q27 BC846, Q28 BC846, Q29 BC846, Q3 BC856, Q30 BC846, Q31 BC846, Q32 BC846, Q33 BC846, Q4 BC856, Q5 BC846, Q6 BC846, Q7 BC856, Q8 BC856, Q9 BC846, U1 MCP2562, U2 STM32F072R, U3 AP3513E, U4 AP1117IE33G, X1 8.000 MHz

Commit message: Adding RGB LED driver
Parts:
- added K1: CONN_3, Sockets_MOLEX_KK-System:Socket_MOLEX-KK-RM2-54mm_Lock_3pin_straight, F.Cu at (238.4, 125.7)
- added Q34: BSS138, Housings_SOT-23_SOT-143_TSOT-6:SOT-23, F.Cu at (233.0, 121.6)
- added R14: 22, Resistors_SMD:R_0603, F.Cu at (231.1, 125.4)
- added R73: 10K, Resistors_SMD:R_0603, F.Cu at (233.7, 124.5)
- added R74: 1K, Resistors_SMD:R_0603, F.Cu at (233.7, 128.3)
- added R75: 22, Resistors_SMD:R_0603, F.Cu at (233.7, 126.4)
- moved R6 11.9 mm to (243.8, 134.3), turned to 180 degrees
- moved R8 10.9 mm to (243.8, 131.8), turned to 180 degrees
- moved I2C1 5.08 mm to (238.4, 135.6)
Connections:
- U2 pad 11: (no net) -> /RGB Output/RGB_DATA
Routing:
- net /RGB Output/RGB_DATA: track 0.00 -> 81.7 mm, vias 0 -> 2
- net +5V: track 342.2 -> 366.9 mm
- net +3.3V: track 303.0 -> 292.4 mm
- net Net-(Q34-Pad3): track 0.00 -> 8.24 mm
- net /Control Logic/SCL: track 103.4 -> 95.2 mm
- net /Control Logic/SDA: track 103.5 -> 98.0 mm
- net Net-(K1-Pad2): track 0.00 -> 4.28 mm
- net Net-(Q34-Pad1): track 0.00 -> 3.73 mm
- net /Control Logic/BOOTLOADER: track 149.4 -> 152.4 mm
- net /Control Logic/~RESET: track 170.3 -> 173.1 mm
- net /Anode Driver/ANODE0: track 86.3 -> 87.3 mm
- net /Anode Driver/ANODE1: track 82.5 -> 83.3 mm
- net /Anode Driver/ANODE2: track 79.0 -> 79.5 mm
- net /Control Logic/SWCLK: track 129.8 -> 130.2 mm, vias 2 -> 3
- net /Control Logic/RXD: track 116.0 -> 116.4 mm, vias 2 -> 3
